File: PCB/Stardance-FlightPad.kicad_pcb (KiCad board)
At the start: 2 copper layers, 79.5 x 81 mm, 21 parts, among them SW1 SW_Push, SW10 RotaryEncoder_Switch, SW11 RotaryEncoder_Switch, SW2 SW_Push, SW3 SW_Push, SW4 SW_Push, SW5 SW_Push, SW6 SW_Push, SW7 SW_Push, SW8 SW_Push, SW9 SW_Push, U1 MOUDLE-SEEEDUINO-XIAO

Commit message: Fixed routing errors in pcb
Routing:
- net Net-(D7-A): track 0.00 -> 12.0 mm
- net Net-(D9-A): track 0.00 -> 12.0 mm
- net Net-(D8-A): track 0.00 -> 12.0 mm
Changed lines of the file:
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@@
+	)
+	(segment
+		(start 74.65 106.96)
+		(end 74.69 107)
+		(width 0.2)
+		(layer "B.Cu")
+		(net "Net-(D8-A)")
+	)
+	(segment
+		(start 74.65 95.04)
+		(end 74.65 106.96)
+		(width 0.2)
+		(layer "B.Cu")
+		(net "Net-(D8-A)")
 	)
 	(segment
@@
 		(layer "F.Cu")
 		(net "/COL2")
+	)
+	(segment
+		(start 93.65 106.96)
+		(end 93.69 107)
+		(width 0.2)
+		(layer "B.Cu")
+		(net "Net-(D9-A)")
+	)
+	(segment
+		(start 93.65 95.04)
+		(end 93.65 106.96)
+		(width 0.2)
+		(layer "B.Cu")
+		(net "Net-(D9-A)")
 	)
 	(segment
@@
 	)
 	(segment
+		(start 55.65 95.04)
+		(end 55.65 106.96)
+		(width 0.2)
+		(layer "B.Cu")
+		(net "Net-(D7-A)")
+	)
+	(segment
+		(start 55.65 106.96)
+		(end 55.69 107)
+		(width 0.2)
+		(layer "B.Cu")
+		(net "Net-(D7-A)")
+	)
+	(segment
